Commit message: 0222

File: src/urdf_demo/urdf/xacro/base.xacro (robot description, xacro)
@@ -9,5 +9,6 @@
 <robot name="my_base" xmlns:xacro="http://www.ros.org/wiki/xacro">
     <!-- 封装变量、常量 -->
-    <xacro:property name="PI" value="3.141"/>
+    <!-- PI 值设置精度需要高一些，否则后续车轮翻转量计算时，可能会出现肉眼不能察觉的车轮倾斜，从而导致模型抖动 -->
+    <xacro:property name="PI" value="3.1415926"/>
     <!-- 宏:黑色设置 -->
     <material name="black">
@@ -19,4 +20,5 @@
     <xacro:property name="base_link_length" value="0.08" /> <!-- base_link 长 -->
     <xacro:property name="earth_space" value="0.015" /> <!-- 离地间距 -->
+    <xacro:property name="base_link_m" value="0.5" /> <!-- 质量  -->
     <!-- 底盘 -->
     <link name="base_footprint">
@@ -37,4 +39,11 @@
         </material>
       </visual>
+      <collision>
+        <geometry>
+          <cylinder radius="${base_link_radius}" length="${base_link_length}" />
+        </geometry>
+        <origin xyz="0 0 0" rpy="0 0 0" />
+      </collision>
+      <xacro:cylinder_inertial_matrix m="${base_link_m}" r="${base_link_radius}" h="${base_link_length}" />
     </link>
     <joint name="base_link2base_footprint" type="fixed">
@@ -43,8 +52,12 @@
       <origin xyz="0 0 ${earth_space + base_link_length / 2 }" />
     </joint>
+    <gazebo reference="base_link">
+        <material>Gazebo/Yellow</material>
+    </gazebo>
     <!-- 驱动轮 -->
     <!-- 驱动轮属性 -->
     <xacro:property name="wheel_radius" value="0.0325" /><!-- 半径 -->
     <xacro:property name="wheel_length" value="0.015" /><!-- 宽度 -->
+    <xacro:property name="wheel_m" value="0.05" /> <!-- 质量  -->
     <!-- 驱动轮宏实现 -->
     <xacro:macro name="add_wheels" params="name flag">
@@ -57,4 +70,11 @@
           <material name="black" />
         </visual>
+        <collision>
+          <geometry>
+            <cylinder radius="${wheel_radius}" length="${wheel_length}" />
+          </geometry>
+          <origin xyz="0.0 0.0 0.0" rpy="${PI / 2} 0.0 0.0" />
+        </collision>
+        <xacro:cylinder_inertial_matrix m="${wheel_m}" r="${wheel_radius}" h="${wheel_length}" />
       </link>
       <joint name="${name}_wheel2base_link" type="continuous">
@@ -64,4 +84,7 @@
         <axis xyz="0 1 0" />
       </joint>
+      <gazebo reference="${name}_wheel">
+        <material>Gazebo/Red</material>
+      </gazebo>
     </xacro:macro>
     <xacro:add_wheels name="left" flag="1" />
@@ -70,4 +93,5 @@
     <!-- 支撑轮属性 -->
     <xacro:property name="support_wheel_radius" value="0.0075" /> <!-- 支撑轮半径 -->
+    <xacro:property name="support_wheel_m" value="0.03" /> <!-- 质量  -->
     <!-- 支撑轮宏 -->
     <xacro:macro name="add_support_wheel" params="name flag" >
@@ -80,4 +104,11 @@
             <material name="black" />
         </visual>
+        <collision>
+            <geometry>
+                <sphere radius="${support_wheel_radius}" />
+            </geometry>
+            <origin xyz="0 0 0" rpy="0 0 0" />
+        </collision>
+        <xacro:sphere_inertial_matrix m="${support_wheel_m}" r="${support_wheel_radius}" />
       </link>
       <joint name="${name}_wheel2base_link" type="continuous">
@@ -87,4 +118,7 @@
           <axis xyz="1 1 1" />
       </joint>
+      <gazebo reference="${name}_wheel">
+        <material>Gazebo/Red</material>
+      </gazebo>
     </xacro:macro>
     <xacro:add_support_wheel name="front" flag="1" />

File: src/urdf_demo/urdf/xacro/camera.xacro (robot description, xacro)
@@ -8,4 +8,5 @@
     <xacro:property name="camera_y" value="0.0" /> <!-- 摄像头安装的y坐标 -->
     <xacro:property name="camera_z" value="${base_link_length / 2 + camera_height / 2}" /> <!-- 摄像头安装的z坐标:底盘高度 / 2 + 摄像头高度 / 2  -->
+    <xacro:property name="camera_m" value="0.01" /> <!-- 摄像头质量 -->
     <!-- 摄像头关节以及link -->
     <link name="camera">
@@ -17,4 +18,11 @@
             <material name="black" />
         </visual>
+        <collision>
+            <geometry>
+                <box size="${camera_length} ${camera_width} ${camera_height}" />
+            </geometry>
+            <origin xyz="0.0 0.0 0.0" rpy="0.0 0.0 0.0" />
+        </collision>
+        <xacro:Box_inertial_matrix m="${camera_m}" l="${camera_length}" w="${camera_width}" h="${camera_height}" />
     </link>
     <joint name="camera2base_link" type="fixed">
@@ -23,3 +31,6 @@
         <origin xyz="${camera_x} ${camera_y} ${camera_z}" />
     </joint>
+    <gazebo reference="camera">
+        <material>Gazebo/Blue</material>
+    </gazebo>
 </robot>

File: src/urdf_demo/urdf/xacro/car.xacro (robot description, xacro)
@@ -1,5 +1,6 @@
 <!-- 组合小车底盘与摄像头与雷达 -->
 <robot name="my_car_camera" xmlns:xacro="http://wiki.ros.org/xacro">
-    <xacro:include filename="demo05_car_base.xacro" />
+    <xacro:include filename="head.xacro" />
+    <xacro:include filename="base.xacro" />
     <xacro:include filename="camera.xacro" />
     <xacro:include filename="lidar.xacro" />

File: src/urdf_demo/urdf/xacro/lidar.xacro (robot description, xacro)
@@ -9,4 +9,5 @@
     <xacro:property name="support_y" value="0.0" /> <!-- 支架安装的y坐标 -->
     <xacro:property name="support_z" value="${base_link_length / 2 + support_length / 2}" /> <!-- 支架安装的z坐标:底盘高度 / 2 + 支架高度 / 2  -->
+    <xacro:property name="support_m" value="0.02" /> <!-- 支架质量 -->
     <link name="support">
         <visual>
@@ -19,4 +20,11 @@
             </material>
         </visual>
+        <collision>
+            <geometry>
+                <cylinder radius="${support_radius}" length="${support_length}" />
+            </geometry>
+            <origin xyz="0.0 0.0 0.0" rpy="0.0 0.0 0.0" />
+        </collision>
+        <xacro:cylinder_inertial_matrix m="${support_m}" r="${support_radius}" h="${support_length}" />
     </link>
     <joint name="support2base_link" type="fixed">
@@ -25,4 +33,7 @@
         <origin xyz="${support_x} ${support_y} ${support_z}" />
     </joint>
+    <gazebo reference="support">
+        <material>Gazebo/White</material>
+    </gazebo>
     <!-- 雷达属性 -->
     <xacro:property name="laser_length" value="0.05" /> <!-- 雷达长度 -->
@@ -31,4 +42,5 @@
     <xacro:property name="laser_y" value="0.0" /> <!-- 雷达安装的y坐标 -->
     <xacro:property name="laser_z" value="${support_length / 2 + laser_length / 2}" /> <!-- 雷达安装的z坐标:支架高度 / 2 + 雷达高度 / 2  -->
+    <xacro:property name="laser_m" value="0.1" /> <!-- 雷达质量 -->
     <!-- 雷达关节以及link -->
     <link name="laser">
@@ -40,4 +52,11 @@
             <material name="black" />
         </visual>
+        <collision>
+            <geometry>
+                <cylinder radius="${laser_radius}" length="${laser_length}" />
+            </geometry>
+            <origin xyz="0.0 0.0 0.0" rpy="0.0 0.0 0.0" />
+        </collision>
+        <xacro:cylinder_inertial_matrix m="${laser_m}" r="${laser_radius}" h="${laser_length}" />
     </link>
     <joint name="laser2support" type="fixed">
@@ -46,3 +65,6 @@
         <origin xyz="${laser_x} ${laser_y} ${laser_z}" />
     </joint>
+    <gazebo reference="laser">
+        <material>Gazebo/Black</material>
+    </gazebo>
 </robot>
